File: LoRa-V3-Sensor-PCB.kicad_pcb (KiCad board)
At the start: 2 copper layers, 10 x 10 mm, 6 parts, among them IC1 BME690, IC2 SHT40-BD1B-R2, IC3 TSL25911FN

Commit message: move ic3 to back side
Parts:
- IC3: moved to B.Cu
- moved IC3 3.26 mm to (150.5, 89.0), turned to 180 degrees
- moved IC1 1.75 mm to (149.0, 89.3)
- moved IC2 1.75 mm to (152.2, 89.3)
- moved C1 1.03 mm to (148.5, 92.0), turned to 0 degrees
- moved C2 1.03 mm to (152.5, 92.0)
Connections:
- CONN1 pad 3: SCL -> SDA
- CONN1 pad 4: SDA -> SCL
- CONN1 pad 5: SDA -> SCL
- CONN1 pad 6: SCL -> SDA
Routing:
- net 3.3V: track 17.0 -> 24.3 mm, vias 2 -> 4
- net SCL: track 11.7 -> 6.63 mm, vias 0 -> 1
- net SDA: track 12.3 -> 15.1 mm, vias 0 -> 1
