File: LoRa-V3-Sensor-PCB.kicad_pcb (KiCad board)
At the start: 2 copper layers, 10 x 10 mm, 6 parts, among them IC1 BME690, IC2 SHT40-BD1B-R2, IC3 TSL25911FN

Commit message: updates bom from schematic to board
Parts:
- IC1: value BME690 -> BME680
- IC2: value SHT40-BD1B-R2 -> SHT45-AD1B-R2
Changed lines of the file:
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@@
 		)
 	)
+	(property "majorVersion" "0")
+	(property "minorVersion" "6")
+	(property "releaseDate" "Wed Oct 15 12:03:39 2025")
+	(property "releaseDateShort" "2025-10-15")
 	(net 0 "")
 	(net 1 "GND")
@@
 			)
 		)
+		(property "mpn" "BC034-08-A-V-0150-L-C"
+			(at 0 0 0)
+			(unlocked yes)
+			(layer "F.Fab")
+			(hide yes)
+			(effects
+				(font
+					(size 1 1)
+					(thickness 0.15)
+				)
+			)
+		)
 		(property ki_fp_filters "Connector*:*_1x??_*")
 		(sheetname "Root")
@@
 			)
 		)
-		(property "Value" "BME690"
+		(property "Value" "BME680"
 			(at 0 2.45 0)
 			(layer "F.Fab")
@@
 			)
 		)
-		(property "manufacturerPartNumber" "BME690"
+		(property "manufacturerPartNumber" "BME680"
+			(at 0 0 0)
+			(unlocked yes)
+			(layer "F.Fab")
+			(hide yes)
+			(effects
+				(font
+					(size 1 1)
+					(thickness 0.15)
+				)
+			)
+		)
+		(property "mpn" "BME680"
 			(at 0 0 0)
 			(unlocked yes)
@@
 			)
 		)
-		(property "Value" "SHT40-BD1B-R2"
+		(property "Value" "SHT45-AD1B-R2"
 			(at 0 2.25 90)
 			(layer "F.Fab")
@@
 			)
 		)
-		(property "manufacturerPartNumber" "SHT40-BD1B-R2"
+		(property "manufacturerPartNumber" "SHT45-AD1B-R2"
 			(at 0 0 -90)
 			(unlocked yes)
@@
 			)
 		)
-		(property "mouserPartNumber" "403-SHT40-AD1F-R2"
+		(property "mpn" "SHT45-AD1B-R2"
 			(at 0 0 -90)
 			(unlocked yes)
@@
 			)
 		)
-		(property "genericPartNumber" "GPC0603104-25-X7R"
+		(property "genericPartNumber" ""
 			(at 0 0 0)
 			(unlocked yes)
@@
 		)
 		(property "manufacturerPartNumber" "CGA3E2X7R1E104K080AA"
+			(at 0 0 0)
+			(unlocked yes)
+			(layer "F.Fab")
+			(hide yes)
+			(effects
+				(font
+					(size 1 1)
+					(thickness 0.15)
+				)
+			)
+		)
+		(property "mpn" "CGA3E2X7R1E104K080AA"
 			(at 0 0 0)
 			(unlocked yes)
@@
 			)
 		)
-		(property "genericPartNumber" "GPC0603104-25-X7R"
+		(property "genericPartNumber" ""
 			(at 0 0 0)
 			(unlocked yes)
@@
 		)
 		(property "manufacturerPartNumber" "CGA3E2X7R1E104K080AA"
+			(at 0 0 0)
+			(unlocked yes)
+			(layer "F.Fab")
+			(hide yes)
+			(effects
+				(font
+					(size 1 1)
+					(thickness 0.15)
+				)
+			)
+		)
+		(property "mpn" "CGA3E2X7R1E104K080AA"
 			(at 0 0 0)
 			(unlocked yes)
@@
 			)
 		)
-		(property "mouserPartNumber" "985-TSL25911FN"
-			(at 0 0 0)
+		(property "mpn" "TSL25911FN"
+			(at 0 0 180)
 			(unlocked yes)
 			(layer "B.Fab")
-			(hide yes)
-			(effects
-				(font
-					(size 1 1)
-					(thickness 0.15)
-				)
-				(justify mirror)
-			)
-		)
-		(property "digikeyPartNumber" "TSL25911FNCT-ND"
-			(at 0 0 0)
-			(unlocked yes)
-			(layer "B.Fab")
